File: bpf.kicad_sch (KiCad schematic)
At the start: 24 parts, among them J81 Conn_Coaxial

Commit message: qrp-fm試作の反映
Parts:
- removed C96: 1p, digikey-footprints:0603, symbol Device:C
- C85, C90: value 1p -> 10p; footprint digikey-footprints:0603 -> Capacitor_THT:C_Disc_D3.4mm_W2.1mm_P2.50mm
- L81, L83: footprint Inductor_SMD:L_Murata_LQH2MCNxxxx02_2.0x1.6mm -> Inductor_SMD:L_0805_2012Metric_Pad1.15x1.40mm_HandSolder
Connections:
- net GND: now also C85.2, C90.2
- net TRXIO: no longer C85.1
- net at C91.2, C92.2, C93.1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: now also C90.1; no longer C90.2
- net at C88.2, C89.2, C91.1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: no longer C90.1
- net at C82.1, C83.1, C84.2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: now also C85.1; no longer C85.2
Other:
- moved on the sheet: C82, C83, C84, C87, L81, L82

Commit message: Add files via upload
秋月の通販コード追加
部品表の代わりにxmlファイルを追加
Parts:
- C81, C83, C85, C86, C89, C90, C92, C94, C98, C99: value 10p -> NM
- C82, C95: value 1p -> 15p
- C84, C97: value 1p -> 6.8p
- C87, C93: value 1p -> NM
- C88, C91: value 1p -> 10p
- L81, L83: value 10n -> 3.3n
- L82, L84: value 1u -> NM
Changed lines of the file:
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@@
       (effects (font (size 1.27 1.27)) (justify left))
     )
-    (property "Value" "1p" (id 1) (at 180.721 96.393 0)
+    (property "Value" "15p" (id 1) (at 180.721 96.393 0)
       (effects (font (size 1.27 1.27)) (justify left))
     )
@@
     (in_bom yes) (on_board yes)
     (property "Reference" "C91" (id 0) (at 146.05 57.0992 90))
-    (property "Value" "1p" (id 1) (at 146.05 59.4106 90))
+    (property "Value" "10p" (id 1) (at 146.05 59.4106 90))
     (property "Footprint" "digikey-footprints:0603" (id 2) (at 149.86 62.5348 0)
       (effects (font (size 1.27 1.27)) hide)
@@
       (effects (font (size 1.27 1.27)) (justify left))
     )
-    (property "Value" "10n" (id 1) (at 191.8462 96.393 0)
+    (property "Value" "3.3n" (id 1) (at 191.8462 96.393 0)
       (effects (font (size 1.27 1.27)) (justify left))
     )
@@
       (effects (font (size 1.27 1.27)) hide)
     )
-    (property "Datasheet" "~" (id 3) (at 190.5 95.25 0)
+    (property "Datasheet" "digikey 0805CS-3N3EJTS" (id 3) (at 190.5 95.25 0)
       (effects (font (size 1.27 1.27)) hide)
     )
@@
       (effects (font (size 1.27 1.27)) (justify left))
     )
-    (property "Value" "10p" (id 1) (at 168.021 96.393 0)
+    (property "Value" "NM" (id 1) (at 168.021 96.393 0)
       (effects (font (size 1.27 1.27)) (justify left))
     )
@@
       (effects (font (size 1.27 1.27)) (justify left))
     )
-    (property "Value" "1p" (id 1) (at 155.321 96.393 0)
+    (property "Value" "NM" (id 1) (at 155.321 96.393 0)
       (effects (font (size 1.27 1.27)) (justify left))
     )
@@
       (effects (font (size 1.27 1.27)) (justify left))
     )
-    (property "Value" "1u" (id 1) (at 204.5462 96.393 0)
+    (property "Value" "NM" (id 1) (at 204.5462 96.393 0)
       (effects (font (size 1.27 1.27)) (justify left))
     )
@@
     (in_bom yes) (on_board yes)
     (property "Reference" "C92" (id 0) (at 146.05 69.7992 90))
-    (property "Value" "10p" (id 1) (at 146.05 72.1106 90))
+    (property "Value" "NM" (id 1) (at 146.05 72.1106 90))
     (property "Footprint" "Capacitor_THT:C_Disc_D3.4mm_W2.1mm_P2.50mm" (id 2) (at 149.86 75.2348 0)
       (effects (font (size 1.27 1.27)) hide)
@@
     (in_bom yes) (on_board yes)
     (property "Reference" "C89" (id 0) (at 120.65 69.7992 90))
-    (property "Value" "10p" (id 1) (at 120.65 72.1106 90))
+    (property "Value" "NM" (id 1) (at 120.65 72.1106 90))
     (property "Footprint" "Capacitor_THT:C_Disc_D3.4mm_W2.1mm_P2.50mm" (id 2) (at 124.46 75.2348 0)
       (effects (font (size 1.27 1.27)) hide)
@@
       (effects (font (size 1.27 1.27)) (justify left))
     )
-    (property "Value" "1p" (id 1) (at 104.521 96.393 0)
+    (property "Value" "NM" (id 1) (at 104.521 96.393 0)
       (effects (font (size 1.27 1.27)) (justify left))
     )
@@
       (effects (font (size 1.27 1.27)) (justify left))
     )
-    (property "Value" "10n" (id 1) (at 115.6462 96.393 0)
+    (property "Value" "3.3n" (id 1) (at 115.6462 96.393 0)
       (effects (font (size 1.27 1.27)) (justify left))
     )
@@
       (effects (font (size 1.27 1.27)) hide)
     )
-    (property "Datasheet" "~" (id 3) (at 114.3 95.25 0)
+    (property "Datasheet" "digikey 0805CS-3N3EJTS" (id 3) (at 114.3 95.25 0)
       (effects (font (size 1.27 1.27)) hide)
     )
@@
       (effects (font (size 1.27 1.27)) (justify left))
     )
-    (property "Value" "10p" (id 1) (at 91.821 96.393 0)
+    (property "Value" "NM" (id 1) (at 91.821 96.393 0)
       (effects (font (size 1.27 1.27)) (justify left))
     )
@@
       (effects (font (size 1.27 1.27)) (justify left))
     )
-    (property "Value" "1p" (id 1) (at 79.121 96.393 0)
+    (property "Value" "15p" (id 1) (at 79.121 96.393 0)
       (effects (font (size 1.27 1.27)) (justify left))
     )
@@
       (effects (font (size 1.27 1.27)) (justify left))
     )
-    (property "Value" "1u" (id 1) (at 128.3462 96.393 0)
+    (property "Value" "NM" (id 1) (at 128.3462 96.393 0)
       (effects (font (size 1.27 1.27)) (justify left))
     )
@@
     (in_bom yes) (on_board yes)
     (property "Reference" "C86" (id 0) (at 82.55 69.7992 90))
-    (property "Value" "10p" (id 1) (at 82.55 72.1106 90))
+    (property "Value" "NM" (id 1) (at 82.55 72.1106 90))
     (property "Footprint" "Capacitor_THT:C_Disc_D3.4mm_W2.1mm_P2.50mm" (id 2) (at 86.36 75.2348 0)
       (effects (font (size 1.27 1.27)) hide)
@@
     (in_bom yes) (on_board yes)
     (property "Reference" "C97" (id 0) (at 196.85 57.0992 90))
-    (property "Value" "1p" (id 1) (at 196.85 59.4106 90))
+    (property "Value" "6.8p" (id 1) (at 196.85 59.4106 90))
     (property "Footprint" "digikey-footprints:0603" (id 2) (at 200.66 62.5348 0)
       (effects (font (size 1.27 1.27)) hide)
@@
     (in_bom yes) (on_board yes)
     (property "Reference" "C98" (id 0) (at 196.85 69.7992 90))
-    (property "Value" "10p" (id 1) (at 196.85 72.1106 90))
+    (property "Value" "NM" (id 1) (at 196.85 72.1106 90))
     (property "Footprint" "Capacitor_THT:C_Disc_D3.4mm_W2.1mm_P2.50mm" (id 2) (at 200.66 75.2348 0)
       (effects (font (size 1.27 1.27)) hide)
@@
       (effects (font (size 1.27 1.27)) (justify left))
     )
-    (property "Value" "10p" (id 1) (at 53.721 83.693 0)
+    (property "Value" "NM" (id 1) (at 53.721 83.693 0)
       (effects (font (size 1.27 1.27)) (justify left))
     )
@@
       (effects (font (size 1.27 1.27)) (justify left))
     )
-    (property "Value" "10p" (id 1) (at 231.521 83.693 0)
+    (property "Value" "NM" (id 1) (at 231.521 83.693 0)
       (effects (font (size 1.27 1.27)) (justify left))
     )
@@
     (in_bom yes) (on_board yes)
     (property "Reference" "C88" (id 0) (at 120.65 57.0992 90))
-    (property "Value" "1p" (id 1) (at 120.65 59.4106 90))
+    (property "Value" "10p" (id 1) (at 120.65 59.4106 90))
     (property "Footprint" "digikey-footprints:0603" (id 2) (at 124.46 62.5348 0)
       (effects (font (size 1.27 1.27)) hide)
@@
     (in_bom yes) (on_board yes)
     (property "Reference" "C84" (id 0) (at 82.55 57.0992 90))
-    (property "Value" "1p" (id 1) (at 82.55 59.4106 90))
+    (property "Value" "6.8p" (id 1) (at 82.55 59.4106 90))
     (property "Footprint" "digikey-footprints:0603" (id 2) (at 86.36 62.5348 0)
       (effects (font (size 1.27 1.27)) hide)
@@
       (effects (font (size 1.27 1.27)) hide)
     )
-    (property "Datasheet" " ~" (id 3) (at 248.92 76.2 0)
+    (property "Datasheet" "C-01422" (id 3) (at 248.92 76.2 0)
       (effects (font (size 1.27 1.27)) hide)
     )
@@
       (effects (font (size 1.27 1.27)) (justify left))
     )
-    (property "Value" "10p" (id 1) (at 67.691 96.393 0)
+    (property "Value" "NM" (id 1) (at 67.691 96.393 0)
       (effects (font (size 1.27 1.27)) (justify left))
     )
@@
       (effects (font (size 1.27 1.27)) (justify left))
     )
-    (property "Value" "10p" (id 1) (at 142.621 96.393 0)
-      (effects (font (size 1.27 1.27)) (justify left))
-    )
+    (property "Value" "NM" (id 1) (at 142.621 96.393 0)
+      (effects (font (size 1.27 1.27)) (justify left))
+    )

Commit message: バンドパスフィルタ見直し
Parts:
- C82: value 15p -> NM
- C83, C90: value NM -> 6p
- C85: value NM -> 12p
- C88: value 10p -> NM
- C89: value NM -> 3.3p
- C91: value 10p -> 3.3p
- C95: value 15p -> 12p
Other:
- company: (none) -> PRUG
- title: (none) -> QRP-TNC
Changed lines of the file:
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@@
 (kicad_sch (version 20211123) (generator eeschema)
   (paper "A4")
+  (title_block
+    (title "QRP-TNC")
+    (date "2022-05-03")
+    (company "PRUG")
+  )
   (junction (at 139.7 76.2) (diameter 0) (color 0 0 0 0)
   )
@@
       (effects (font (size 1.27 1.27)) (justify left))
     )
-    (property "Value" "15p" (id 1) (at 180.721 96.393 0)
+    (property "Value" "12p" (id 1) (at 180.721 96.393 0)
       (effects (font (size 1.27 1.27)) (justify left))
     )
@@
     (in_bom yes) (on_board yes)
     (property "Reference" "C91" (id 0) (at 146.05 57.0992 90))
-    (property "Value" "10p" (id 1) (at 146.05 59.4106 90))
+    (property "Value" "3.3p" (id 1) (at 146.05 59.4106 90))
     (property "Footprint" "digikey-footprints:0603" (id 2) (at 149.86 62.5348 0)
       (effects (font (size 1.27 1.27)) hide)
@@
     (in_bom yes) (on_board yes)
     (property "Reference" "C89" (id 0) (at 120.65 69.7992 90))
-    (property "Value" "NM" (id 1) (at 120.65 72.1106 90))
+    (property "Value" "3.3p" (id 1) (at 120.65 72.1106 90))
     (property "Footprint" "Capacitor_THT:C_Disc_D3.4mm_W2.1mm_P2.50mm" (id 2) (at 124.46 75.2348 0)
       (effects (font (size 1.27 1.27)) hide)
@@
       (effects (font (size 1.27 1.27)) (justify left))
     )
-    (property "Value" "NM" (id 1) (at 91.821 96.393 0)
+    (property "Value" "6p" (id 1) (at 91.821 96.393 0)
       (effects (font (size 1.27 1.27)) (justify left))
     )
@@
       (effects (font (size 1.27 1.27)) (justify left))
     )
-    (property "Value" "15p" (id 1) (at 79.121 96.393 0)
+    (property "Value" "NM" (id 1) (at 79.121 96.393 0)
       (effects (font (size 1.27 1.27)) (justify left))
     )
@@
     (in_bom yes) (on_board yes)
     (property "Reference" "C88" (id 0) (at 120.65 57.0992 90))
-    (property "Value" "10p" (id 1) (at 120.65 59.4106 90))
+    (property "Value" "NM" (id 1) (at 120.65 59.4106 90))
     (property "Footprint" "digikey-footprints:0603" (id 2) (at 124.46 62.5348 0)
       (effects (font (size 1.27 1.27)) hide)
@@
       (effects (font (size 1.27 1.27)) (justify left))
     )
-    (property "Value" "NM" (id 1) (at 67.691 96.393 0)
+    (property "Value" "12p" (id 1) (at 67.691 96.393 0)
       (effects (font (size 1.27 1.27)) (justify left))
     )
@@
       (effects (font (size 1.27 1.27)) (justify left))
     )
-    (property "Value" "NM" (id 1) (at 142.621 96.393 0)
-      (effects (font (size 1.27 1.27)) (justify left))
-    )
+    (property "Value" "6p" (id 1) (at 142.621 96.393 0)
+      (effects (font (size 1.27 1.27)) (justify left))
+    )
