File: fm-tnc.kicad_pcb (KiCad board)
At the start: 2 copper layers, 100 x 68 mm, 97 parts, among them IC11 NM(TO220), IC12 NJM2845DL1-33, IC31 BK4802P, J11 Conn_01x03, J12 Conn_01x06_Female, J13 Conn_01x09_Female, J14 Conn_01x07_Socket, J15 Conn_01x07_Socket, J16 Conn_01x06_Female, J17 Conn_01x08_Female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

Commit message: Add files via upload
Parts:
- C19: value 0.1u -> 1u
- C21: value 1u -> NM
- C31, C36, C38: value 1u -> 0.1u
- C35: value 27p -> 22p
- C39: value 27p -> 33p
- C45: value NM -> 0.1u
- C52, C54: value 4p -> 22p
- C53: value 22p -> 18p
- J17: value Conn_01x08_Female -> Conn_01x06_Female; footprint Connector_PinHeader_2.54mm:PinHeader_1x08_P2.54mm_Vertical -> UserLib:PinHeader_1x06_P2.54mm_Vertical
- L51, L52: value 50n -> 20n
- R25: value NM -> 10k
- R34: value 10k -> NM
- moved J17 17.8 mm to (127.0, 68.6), turned to 180 degrees
- moved R25 11.4 mm to (116.8, 40.6), turned to 180 degrees
Connections:
- net /cpu/M5_3.3V renamed /cpu/LMT_3.3V
- J17 pad 1: Net-(J17-Pin_1) -> GND
- J17 pad 2: GND -> /cpu/M5_IO0
- J17 pad 3: Net-(J15-Pin_3) -> /cpu/M5_EN
- J17 pad 4: /cpu/M5_TXD -> /cpu/M5_RXD
- J17 pad 5: /cpu/M5_RXD -> /cpu/M5_TXD
- J17 pad 6: /cpu/M5_EN -> Net-(J15-Pin_3)
- R25 pad 1: +5V -> Net-(J15-Pin_3)
- R25 pad 2: Net-(J17-Pin_1) -> /cpu/M5_P25
Routing:
- net M5_ADC: track 227.9 -> 161.2 mm, vias 6 -> 1
- net GND: track 586.7 -> 645.4 mm, vias 144 -> 147
- net Net-(J17-Pin_1): track 2.54 -> 0.00 mm
- net Net-(J15-Pin_3): track 64.7 -> 67.3 mm

Commit message: CAD data update
CADデータを更新
Parts:
- removed R12, R20: 0, Resistor_THT:R_Axial_DIN0207_L6.3mm_D2.5mm_P2.54mm_Vertical
- removed TP31: NM, usr-Library:PinHeader_1x01
- added C10: 100u, Capacitor_THT:CP_Radial_D4.0mm_P2.00mm, F.Cu at (108.6, 96.5)
- added C57: NM, Capacitor_THT:C_Disc_D3.4mm_W2.1mm_P2.50mm, F.Cu at (55.9, 61.0)
- added R27: NM, Resistor_THT:R_Axial_DIN0207_L6.3mm_D2.5mm_P2.54mm_Vertical, F.Cu at (53.3, 86.4)
- C18: value 1000p -> 0.01u
- Q11: value NM(DTC114E) -> NM(DTC143E)
- R26: value 10k -> 4.7k
- X31: value Crystal -> 21.250
- moved J17 12.7 mm to (127.0, 55.9), turned to 0 degrees
- moved J19 7.62 mm to (83.8, 63.5), turned to 180 degrees
- moved C16 2.54 mm to (94.0, 58.4), turned to 90 degrees
- moved R14 2.54 mm to (78.7, 58.4)
- moved C54 2.52 mm to (55.9, 55.9)
- moved C43 1.25 mm to (50.8, 76.8), turned to 90 degrees
- moved G*** 0.64 mm to (41.9, 87.0)
Connections:
- C13 pad 1: /cpu/+3.3V-REG -> +3V3
- C16 pad 1: Net-(J12-Pin_1) -> /cpu/LMT_3.3V
- C43 pad 1: Net-(C43-Pad1) -> /trx/SPK
- IC11 pad 3: /cpu/+3.3V-REG -> +3V3
- IC12 pad 3: /cpu/+3.3V-REG -> +3V3
- IC31 pad 10: Net-(IC31-EARON) -> unconnected-(IC31-EARON-Pad10)
- J12 pad 1: Net-(J12-Pin_1) -> /cpu/LMT_3.3V
- J14 pad 4: TNC_LED -> unconnected-(J14-Pin_4-Pad4)
- J17 pad 1: GND -> Net-(J15-Pin_3)
- J17 pad 2: /cpu/M5_IO0 -> /cpu/M5_TXD
- J17 pad 3: /cpu/M5_EN -> /cpu/M5_RXD
- J17 pad 4: /cpu/M5_RXD -> /cpu/M5_EN
- J17 pad 5: /cpu/M5_TXD -> /cpu/M5_IO0
- J17 pad 6: Net-(J15-Pin_3) -> GND
- J19 pad 1: GND -> M5_SCL
- J19 pad 2: Net-(J12-Pin_1) -> M5_SDA
- J19 pad 3: Net-(J12-Pin_3) -> /cpu/LMT_3.3V
- J19 pad 4: M5_SDA -> GND
- J31 pad 2: M5_ADC -> /trx/SPK
- R35 pad 2: Net-(C43-Pad1) -> /trx/SPK
Routing:
- net GND: track 645.4 -> 617.6 mm, vias 147 -> 149
- net /trx/SPK: track 0.00 -> 23.2 mm
- net M5_SDA: track 122.1 -> 140.8 mm, vias 3 -> 2
- net Net-(J12-Pin_1): track 17.3 -> 0.00 mm
- net Net-(C43-Pad1): track 16.4 -> 0.00 mm
- net M5_SCL: track 110.9 -> 124.5 mm
- net /cpu/+3.3V-REG: track 6.91 -> 0.00 mm
- net +3V3: track 87.6 -> 93.0 mm
- net Net-(IC31-EARON): track 5.31 -> 0.00 mm
- net Net-(J12-Pin_3): track 16.2 -> 11.1 mm
- net /cpu/LMT_3.3V: track 76.7 -> 73.1 mm
- net Net-(C54-Pad2): track 4.93 -> 7.51 mm
- net M5_ADC: track 161.2 -> 163.0 mm, vias 1 -> 2
Other:
- board text added: "21.250M"
- board text added: "3V"
- board text added: "5V"
- board text added: "B"
- board text added: "BK4802P"
- board text added: "BOOT"
- board text added: "C"
- board text added: "CHK"
- board text added: "D"
- board text added: "DCD"
- board text added: "E"
- board text added: "G"
- board text added: "I"
- board text added: "JK1MLY 2023.7"
- board text added: "M"
- board text added: "O"
- board text added: "P"
- board text added: "RF"
- board text added: "RX"
- board text added: "S"
- board text added: "SCL"
- board text added: "SDA"
- board text added: "TX"
- board text added: "V"
- board text removed: "G18"
- board text removed: "G19"
- board text removed: "G25"
- board text removed: "JK1MLY 2023.6"
