File: trx.kicad_sch (KiCad schematic)
At the start: 28 parts, among them IC31 BK4802P, IC32 PIC12LF1501-IP, J31 Conn_01x04_Male, J32 Conn_01x06_Male, X31 Crystal

Commit message: qrp-fm試作の反映
Parts:
- C32, C44: value 0.1u -> NM
- C34: value 10u -> 470u; footprint Capacitor_THT:CP_Radial_Tantal_D7.0mm_P2.50mm -> Capacitor_THT:CP_Radial_D8.0mm_P2.50mm
- C35, C39: value 15p -> 27p
- C43: footprint Capacitor_THT:CP_Radial_Tantal_D5.0mm_P2.50mm -> Capacitor_THT:CP_Radial_D5.0mm_P2.00mm
- D31: value LED -> NM(LED)
- IC32: value PIC12LF1501-IP -> NM(PIC12LF1501-IP)
- J31: value Conn_01x04_Male -> NM
- R32, R33, R37: value 1k -> NM
- R34: value 1k -> 10k
- R35: value 1k -> 10
- R36: value 1k -> nM
Other:
- note added: "PICKit(IC32) Debug(IC31)"
- note added: "Ver2022.2 Jumper C14 - R13(+3.3V)"
Changed lines of the file:
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@@
     (stroke (width 0) (type default) (color 0 0 0 0))
+  )
+  (text "Ver2022.2 Jumper\nC14 - R13(+3.3V)" (at 44.45 44.45 0)
+    (effects (font (size 1.27 1.27)) (justify left bottom))
+  )
+  (text "PICKit(IC32)\nDebug(IC31)" (at 242.57 66.04 0)
+    (effects (font (size 1.27 1.27)) (justify left bottom))
   )
   (label "PTT" (at 96.52 105.41 0)
@@
     (in_bom yes) (on_board yes)
     (property "Reference" "D31" (id 0) (at 240.2078 99.8982 0))
-    (property "Value" "LED" (id 1) (at 240.2078 102.2096 0))
+    (property "Value" "NM(LED)" (id 1) (at 240.2078 102.2096 0))
     (property "Footprint" "digikey-footprints:LED_3mm_Radial" (id 2) (at 240.03 105.41 0)
       (effects (font (size 1.27 1.27)) hide)
@@
     (in_bom yes) (on_board yes)
     (property "Reference" "IC32" (id 0) (at 187.96 90.17 0))
-    (property "Value" "PIC12LF1501-IP" (id 1) (at 195.58 107.95 0))
+    (property "Value" "NM(PIC12LF1501-IP)" (id 1) (at 182.88 115.57 0))
     (property "Footprint" "Package_SO:SOP-8_3.9x4.9mm_P1.27mm" (id 2) (at 196.85 86.36 0)
       (effects (font (size 1.27 1.27)) (justify left) hide)
@@
     (in_bom yes) (on_board yes)
     (property "Reference" "R34" (id 0) (at 170.18 41.7322 90))
-    (property "Value" "1k" (id 1) (at 170.18 44.0436 90))
+    (property "Value" "10k" (id 1) (at 170.18 44.0436 90))
     (property "Footprint" "Resistor_THT:R_Axial_DIN0207_L6.3mm_D2.5mm_P2.54mm_Vertical" (id 2) (at 170.18 48.768 90)
       (effects (font (size 1.27 1.27)) hide)
@@
       (effects (font (size 1.27 1.27)) (justify left))
     )
-    (property "Value" "15p" (id 1) (at 114.681 76.073 0)
+    (property "Value" "27p" (id 1) (at 114.681 76.073 0)
       (effects (font (size 1.27 1.27)) (justify left))
     )
@@
       (effects (font (size 1.27 1.27)) (justify left))
     )
-    (property "Value" "15p" (id 1) (at 135.001 76.073 0)
+    (property "Value" "27p" (id 1) (at 135.001 76.073 0)
       (effects (font (size 1.27 1.27)) (justify left))
     )
@@
       (effects (font (size 1.27 1.27)) (justify left))
     )
-    (property "Value" "0.1u" (id 1) (at 215.011 88.773 0)
+    (property "Value" "NM" (id 1) (at 215.011 88.773 0)
       (effects (font (size 1.27 1.27)) (justify left))
     )
@@
     (in_bom yes) (on_board yes)
     (property "Reference" "R36" (id 0) (at 229.87 100.1522 90))
-    (property "Value" "1k" (id 1) (at 229.87 102.4636 90))
+    (property "Value" "nM" (id 1) (at 229.87 102.4636 90))
     (property "Footprint" "Resistor_THT:R_Axial_DIN0207_L6.3mm_D2.5mm_P2.54mm_Vertical" (id 2) (at 229.87 107.188 90)
       (effects (font (size 1.27 1.27)) hide)
@@
     (in_bom yes) (on_board yes)
     (property "Reference" "R35" (id 0) (at 187.96 35.3822 90))
-    (property "Value" "1k" (id 1) (at 187.96 37.6936 90))
+    (property "Value" "10" (id 1) (at 187.96 37.6936 90))
     (property "Footprint" "Resistor_THT:R_Axial_DIN0207_L6.3mm_D2.5mm_P2.54mm_Vertical" (id 2) (at 187.96 42.418 90)
       (effects (font (size 1.27 1.27)) hide)
@@
       (effects (font (size 1.27 1.27)) (justify left))
     )
-    (property "Value" "0.1u" (id 1) (at 104.521 97.663 0)
+    (property "Value" "NM" (id 1) (at 104.521 97.663 0)
       (effects (font (size 1.27 1.27)) (justify left))
     )
@@
     (property "Reference" "C43" (id 0) (at 196.85 34.163 90))
     (property "Value" "10u" (id 1) (at 196.85 36.4744 90))
-    (property "Footprint" "Capacitor_THT:CP_Radial_Tantal_D5.0mm_P2.50mm" (id 2) (at 200.66 39.6748 0)
+    (property "Footprint" "Capacitor_THT:CP_Radial_D5.0mm_P2.00mm" (id 2) (at 200.66 39.6748 0)
       (effects (font (size 1.27 1.27)) hide)
     )
@@
       (effects (font (size 1.27 1.27)) (justify left))
     )
-    (property "Value" "1k" (id 1) (at 116.078 97.663 0)
+    (property "Value" "NM" (id 1) (at 116.078 97.663 0)
       (effects (font (size 1.27 1.27)) (justify left))
     )
@@
     (in_bom yes) (on_board yes)
     (property "Reference" "R37" (id 0) (at 218.44 55.7022 90))
-    (property "Value" "1k" (id 1) (at 218.44 58.0136 90))
+    (property "Value" "NM" (id 1) (at 218.44 58.0136 90))
     (property "Footprint" "Resistor_THT:R_Axial_DIN0207_L6.3mm_D2.5mm_P2.54mm_Vertical" (id 2) (at 218.44 62.738 90)
       (effects (font (size 1.27 1.27)) hide)
@@
       (effects (font (size 1.27 1.27)) (justify right))
     )
-    (property "Value" "Conn_01x04_Male" (id 1) (at 83.1088 108.3818 0)
+    (property "Value" "NM" (id 1) (at 83.1088 108.3818 0)
       (effects (font (size 1.27 1.27)) (justify right))
     )
@@
     (pin "4")
   )
-  (symbol (lib_id "Device:CP") (at 82.55 43.18 0)
+  (symbol (lib_id "Device:CP") (at 82.55 43.18 0) (unit 1)
     (in_bom yes) (on_board yes)
     (property "Reference" "C34" (id 0) (at 85.5472 42.0116 0)
       (effects (font (size 1.27 1.27)) (justify left))
     )
-    (property "Value" "10u" (id 1) (at 85.5472 44.323 0)
-      (effects (font (size 1.27 1.27)) (justify left))
-    )
-    (property "Footprint" "Capacitor_THT:CP_Radial_Tantal_D7.0mm_P2.50mm" (id 2) (at 83.5152 46.99 0)
+    (property "Value" "470u" (id 1) (at 85.5472 44.323 0)
+      (effects (font (size 1.27 1.27)) (justify left))
+    )
+    (property "Footprint" "Capacitor_THT:CP_Radial_D8.0mm_P2.50mm" (id 2) (at 83.5152 46.99 0)
       (effects (font (size 1.27 1.27)) hide)
     )
@@
       (effects (font (size 1.27 1.27)) (justify left))
     )
-    (property "Value" "1k" (id 1) (at 95.758 96.393 0)
-      (effects (font (size 1.27 1.27)) (justify left))
-    )
+    (property "Value" "NM" (id 1) (at 95.758 96.393 0)
+      (effects (font (size 1.27 1.27)) (justify left))
+    )

Commit message: Add files via upload
秋月の通販コード追加
部品表の代わりにxmlファイルを追加
Parts:
- R36: value nM -> NM
- TP31: value TestPoint -> NM
Changed lines of the file:
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@@
       (effects (font (size 1.27 1.27)) hide)
     )
-    (property "Datasheet" "http://www.bekencorp.com/en/goods/detail/cid/19.html" (id 3) (at 143.51 57.15 0)
+    (property "Datasheet" "aitendo" (id 3) (at 143.51 57.15 0)
       (effects (font (size 1.27 1.27)) hide)
     )
@@
       (effects (font (size 1.27 1.27)) hide)
     )
-    (property "Datasheet" "~" (id 3) (at 127 69.85 0)
+    (property "Datasheet" "aitendo" (id 3) (at 127 69.85 0)
       (effects (font (size 1.27 1.27)) hide)
     )
@@
       (effects (font (size 1.27 1.27)) hide)
     )
-    (property "Datasheet" "~" (id 3) (at 240.03 105.41 0)
+    (property "Datasheet" "I-11577" (id 3) (at 240.03 105.41 0)
       (effects (font (size 1.27 1.27)) hide)
     )
@@
       (effects (font (size 1.27 1.27)) (justify left) hide)
     )
-    (property "Datasheet" "http://ww1.microchip.com/downloads/en/DeviceDoc/41615A.pdf" (id 3) (at 195.58 102.87 0)
+    (property "Datasheet" "I-02114" (id 3) (at 195.58 102.87 0)
       (effects (font (size 1.27 1.27)) hide)
     )
@@
       (effects (font (size 1.27 1.27)) hide)
     )
-    (property "Datasheet" "~" (id 3) (at 115.57 49.53 0)
+    (property "Datasheet" "P-15940" (id 3) (at 115.57 49.53 0)
       (effects (font (size 1.27 1.27)) hide)
     )
@@
       (effects (font (size 1.27 1.27)) hide)
     )
-    (property "Datasheet" "~" (id 3) (at 156.21 74.93 0)
+    (property "Datasheet" "P-15940" (id 3) (at 156.21 74.93 0)
       (effects (font (size 1.27 1.27)) hide)
     )
@@
       (effects (font (size 1.27 1.27)) hide)
     )
-    (property "Datasheet" "~" (id 3) (at 165.1 74.93 0)
+    (property "Datasheet" "P-15940" (id 3) (at 165.1 74.93 0)
       (effects (font (size 1.27 1.27)) hide)
     )
@@
       (effects (font (size 1.27 1.27)) hide)
     )
-    (property "Datasheet" "~" (id 3) (at 69.85 43.18 0)
+    (property "Datasheet" "P-15940" (id 3) (at 69.85 43.18 0)
       (effects (font (size 1.27 1.27)) hide)
     )
@@
       (effects (font (size 1.27 1.27)) hide)
     )
-    (property "Datasheet" "~" (id 3) (at 127 46.99 0)
+    (property "Datasheet" "P-15940" (id 3) (at 127 46.99 0)
       (effects (font (size 1.27 1.27)) hide)
     )
@@
       (effects (font (size 1.27 1.27)) hide)
     )
-    (property "Datasheet" "~" (id 3) (at 104.14 52.07 0)
+    (property "Datasheet" "P-15940" (id 3) (at 104.14 52.07 0)
       (effects (font (size 1.27 1.27)) hide)
     )
@@
     (in_bom yes) (on_board yes)
     (property "Reference" "R36" (id 0) (at 229.87 100.1522 90))
-    (property "Value" "nM" (id 1) (at 229.87 102.4636 90))
+    (property "Value" "NM" (id 1) (at 229.87 102.4636 90))
     (property "Footprint" "Resistor_THT:R_Axial_DIN0207_L6.3mm_D2.5mm_P2.54mm_Vertical" (id 2) (at 229.87 107.188 90)
       (effects (font (size 1.27 1.27)) hide)
@@
       (effects (font (size 1.27 1.27)) hide)
     )
-    (property "Datasheet" "~" (id 3) (at 120.65 74.93 0)
+    (property "Datasheet" "P-15470" (id 3) (at 120.65 74.93 0)
       (effects (font (size 1.27 1.27)) hide)
     )
@@
       (effects (font (size 1.27 1.27)) hide)
     )
-    (property "Datasheet" "~" (id 3) (at 64.77 36.83 0)
+    (property "Datasheet" "R-25000" (id 3) (at 64.77 36.83 0)
       (effects (font (size 1.27 1.27)) hide)
     )
@@
       (effects (font (size 1.27 1.27)) (justify left))
     )
-    (property "Value" "TestPoint" (id 1) (at 193.7258 58.2168 0)
+    (property "Value" "NM" (id 1) (at 193.7258 58.2168 0)
       (effects (font (size 1.27 1.27)) (justify left))
     )
@@
       (effects (font (size 1.27 1.27)) hide)
     )
-    (property "Datasheet" "~" (id 3) (at 237.49 66.04 0)
+    (property "Datasheet" "C-00167" (id 3) (at 237.49 66.04 0)
       (effects (font (size 1.27 1.27)) hide)
     )
@@
       (effects (font (size 1.27 1.27)) hide)
     )
-    (property "Datasheet" "~" (id 3) (at 83.82 105.41 0)
-      (effects (font (size 1.27 1.27)) hide)
-    )
+    (property "Datasheet" "C-00167" (id 3) (at 83.82 105.41 0)
+      (effects (font (size 1.27 1.27)) hide)
+    )

Commit message: バンドパスフィルタ見直し
Other:
- company: (none) -> PRUG
- title: (none) -> QRP-TNC
Changed lines of the file:
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@@
 (kicad_sch (version 20211123) (generator eeschema)
   (paper "A4")
+  (title_block
+    (title "QRP-TNC")
+    (date "2022-05-03")
+    (company "PRUG")
+  )
   (junction (at 173.99 68.58) (diameter 0) (color 0 0 0 0)
   )

Commit message: Add files via upload
Parts:
- removed C44: NM, Capacitor_THT:C_Disc_D3.4mm_W2.1mm_P2.50mm, symbol Device:C
- removed D31: NM(LED), digikey-footprints:LED_3mm_Radial, symbol Device:LED
- removed IC32: NM(PIC12LF1501-IP), Package_SO:SOP-8_3.9x4.9mm_P1.27mm, symbol MCU_Microchip_PIC12:PIC12LF1501-IP
- removed J32: Conn_01x06_Male, Connector_PinHeader_2.54mm:PinHeader_1x06_P2.54mm_Vertical, symbol Connector:Conn_01x06_Male
- removed R36, R37: NM, Resistor_THT:R_Axial_DIN0207_L6.3mm_D2.5mm_P2.54mm_Vertical, symbol Device:R
- removed TP31: NM, Connector_PinHeader_2.54mm:PinHeader_1x01_P2.54mm_Vertical, symbol Connector:TestPoint
- added C45: 0.1u, Capacitor_THT:C_Disc_D3.4mm_W2.1mm_P2.50mm, symbol Device:C
- added C51, C55: 10p, Capacitor_THT:C_Disc_D3.4mm_W2.1mm_P2.50mm, symbol Device:C
- added C52, C54: 22p, Capacitor_THT:C_Disc_D3.4mm_W2.1mm_P2.50mm, symbol Device:C
- added C53: 18p, Capacitor_THT:C_Disc_D3.4mm_W2.1mm_P2.50mm, symbol Device:C
- added C56, C57: NM, Capacitor_THT:C_Disc_D3.4mm_W2.1mm_P2.50mm, symbol Device:C
- added J51: Conn_Coaxial, digikey-footprints:RF_SMA_Vertical_5-1814832-1, symbol usr_Library:Conn_Coaxial1
- added L51, L52: 20n, usr-Library:coil3_7mm, symbol Device:L
- added R27: NM, Resistor_THT:R_Axial_DIN0207_L6.3mm_D2.5mm_P2.54mm_Vertical, symbol Device:R
- added R38, R39: 3.3k, Resistor_THT:R_Axial_DIN0207_L6.3mm_D2.5mm_P2.54mm_Vertical, symbol Device:R
- C31, C36, C38: value 1u -> 0.1u
- C34: footprint Capacitor_THT:CP_Radial_D8.0mm_P2.50mm -> Capacitor_THT:CP_Radial_D8.0mm_P3.50mm
- C35: value 27p -> 22p
- C37: value 10p -> 30p
- C40: value 100p -> 1000p
- R34: value 10k -> NM
- X31: value Crystal -> 21.250
Connections:
- net +3.3V-TR: no longer R32.1
- net +3V3: now also C45.1, R38.1, R39.1
- net GND: now also C45.2, C51.2, C53.1, C55.2, C56.2, C57.2, J51.1 (G), R27.1
- net M5_SCL: now also R39.2
- net M5_SDA: now also R38.2
- net MIC: now also R32.1
- net TNC_IN: no longer J31.3 (Pin_3)
- net SPK: now reaches C43.1, R35.2
- net SPK: now also J31.2 (Pin_2), R27.2
- net PTT renamed TNC_PTT
- net TNC_PTT: now also J31.3 (Pin_3); no longer J31.2 (Pin_2)
- net TRXIO: no longer names the net of C40.2
- net TRXIO: now also C51.1, L51.1
- new net: C52.1, C56.1, L51.2
- new net: C55.1, J51.2 (S), L52.2
- new net: C52.2, C53.2, C54.1
- new net: C54.2, C57.1, L52.1
Other:
- note added: "5mm 1.5T"
- note added: "R32 Yaesu 2.2k Standard 22k ICOM 22k KENWOOD open"
- note removed: "PICKit(IC32) Debug(IC31)"
- note removed: "Ver2022.2 Jumper C14 - R13(+3.3V)"
- company: PRUG -> PRUG / JK1MLY
- moved on the sheet: C31, C32, C33, C34, C35, C36, C37, C38, C39, C40, C41, C42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
